File: board.sch (EAGLE design)
At the start: 34 parts, among them U1 MCP73831

Commit message: lipo-chg in place (I hope)
Parts:
- removed R1: 100k, rcl:R-US_R0805
- removed R2: 50k, rcl:R-US_R0805
- added C4: 4.7uF, rcl:C-EUC0805
- added LED1: (no value), led:LEDCHIP-LED0603
- added RSENSHI: 100k, rcl:R-US_R0603
- added RSENSLO: 50k, rcl:R-US_R0603
- added RSTATLED: 330, rcl:R-US_R0603
Connections:
- removed net VBAT_SENSE: C1.1, R1.1, R2.2
- new net N$2: LED1.C, U1.STAT
- new net N$3: LED1.A, RSTATLED.1
- new net PD5: PORTD.6
- net GND: now also C4.1, RSENSLO.2; no longer R2.1
- net PB0/XMEGA_AREF: now also RPROG1.2
- net PB1/VBAT_SENSE: now also C1.1, RSENSHI.2, RSENSLO.1
- net PD5/CHGCTRL: no longer PORTD.6, RPROG1.2
- net VBAT: now also C4.2, RSENSHI.1; no longer R1.2
- net VXMEGA_USB: now also RSTATLED.2
Changed lines of the file:
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@@
 <part name="BAT" library="SparkFun-Connectors" deviceset="JST_2MM_MALE" device=""/>
 <part name="BAT_ALT" library="SparkFun-Connectors" deviceset="M02" device="PTH"/>
-<part name="R1" library="rcl" deviceset="R-US_" device="R0805" value="100k"/>
-<part name="R2" library="rcl" deviceset="R-US_" device="R0805" value="50k"/>
 <part name="GND6" library="supply1" deviceset="GND" device=""/>
 <part name="P+2" library="supply1" deviceset="V+" device=""/>
@@
 <part name="RPROG1" library="rcl" deviceset="R-US_" device="R0603" value="2.8k"/>
 <part name="GND10" library="supply1" deviceset="GND" device=""/>
+<part name="C4" library="rcl" deviceset="C-EU" device="C0805" value="4.7uF"/>
+<part name="GND11" library="supply1" deviceset="GND" device=""/>
+<part name="RSTATLED" library="rcl" deviceset="R-US_" device="R0603" value="330"/>
+<part name="LED1" library="led" deviceset="LED" device="CHIP-LED0603"/>
+<part name="RSENSHI" library="rcl" deviceset="R-US_" device="R0603" value="100k"/>
+<part name="RSENSLO" library="rcl" deviceset="R-US_" device="R0603" value="50k"/>
 </parts>
 <sheets>
@@
 <instance part="BAT" gate="G$1" x="-12.7" y="55.88" rot="R90"/>
 <instance part="BAT_ALT" gate="G$1" x="-15.24" y="45.72"/>
-<instance part="R1" gate="G$1" x="-27.94" y="114.3" rot="R90"/>
-<instance part="R2" gate="G$1" x="-27.94" y="101.6" rot="R90"/>
 <instance part="GND6" gate="1" x="-27.94" y="91.44"/>
 <instance part="P+2" gate="1" x="-27.94" y="124.46"/>
@@
 <instance part="RPROG1" gate="G$1" x="5.08" y="20.32" rot="R270"/>
 <instance part="GND10" gate="1" x="-5.08" y="12.7"/>
+<instance part="C4" gate="G$1" x="-15.24" y="33.02"/>
+<instance part="GND11" gate="1" x="-17.78" y="35.56" rot="R270"/>
+<instance part="RSTATLED" gate="G$1" x="-35.56" y="7.62" rot="R270"/>
+<instance part="LED1" gate="G$1" x="-35.56" y="17.78" rot="R180"/>
+<instance part="RSENSHI" gate="G$1" x="-27.94" y="114.3" rot="R270"/>
+<instance part="RSENSLO" gate="G$1" x="-27.94" y="101.6" rot="R270"/>
 </instances>
 <busses>
@@
 </segment>
 <segment>
-<pinref part="R2" gate="G$1" pin="1"/>
 <pinref part="GND6" gate="1" pin="GND"/>
 <wire x1="-27.94" y1="93.98" x2="-27.94" y2="96.52" width="0.1524" layer="91"/>
@@
 <wire x1="-27.94" y1="93.98" x2="-22.86" y2="93.98" width="0.1524" layer="91"/>
 <wire x1="-22.86" y1="93.98" x2="-22.86" y2="99.06" width="0.1524" layer="91"/>
+<pinref part="RSENSLO" gate="G$1" pin="2"/>
 </segment>
 <segment>
@@
 <pinref part="GND10" gate="1" pin="GND"/>
 </segment>
+<segment>
+<pinref part="C4" gate="G$1" pin="1"/>
+<pinref part="GND11" gate="1" pin="GND"/>
+</segment>
 </net>
 <net name="VBAT" class="1">
@@
 <segment>
 <pinref part="P+2" gate="1" pin="V+"/>
-<pinref part="R1" gate="G$1" pin="2"/>
 <wire x1="-27.94" y1="121.92" x2="-27.94" y2="119.38" width="0.1524" layer="91"/>
+<pinref part="RSENSHI" gate="G$1" pin="1"/>
 </segment>
 <segment>
@@
 <pinref part="U1" gate="G$1" pin="VBAT"/>
 <wire x1="-15.24" y1="27.94" x2="-10.16" y2="27.94" width="0.1524" layer="91"/>
+<pinref part="C4" gate="G$1" pin="2"/>
+<junction x="-15.24" y="27.94"/>
 </segment>
 </net>
@@
 <pinref part="U1" gate="G$1" pin="VIN"/>
 <wire x1="-35.56" y1="27.94" x2="-40.64" y2="27.94" width="0.1524" layer="91"/>
+<pinref part="RSTATLED" gate="G$1" pin="2"/>
+<wire x1="-35.56" y1="2.54" x2="-40.64" y2="2.54" width="0.1524" layer="91"/>
+<wire x1="-40.64" y1="2.54" x2="-40.64" y2="27.94" width="0.1524" layer="91"/>
+<wire x1="-40.64" y1="27.94" x2="-43.18" y2="27.94" width="0.1524" layer="91"/>
+<junction x="-40.64" y="27.94"/>
 </segment>
 </net>
@@
 </segment>
 </net>
-<net name="VBAT_SENSE" class="0">
-<segment>
-<pinref part="R1" gate="G$1" pin="1"/>
-<pinref part="R2" gate="G$1" pin="2"/>
-<wire x1="-27.94" y1="106.68" x2="-27.94" y2="109.22" width="0.1524" layer="91"/>
-<pinref part="C1" gate="G$1" pin="1"/>
-<wire x1="-22.86" y1="106.68" x2="-27.94" y2="106.68" width="0.1524" layer="91"/>
-<junction x="-27.94" y="106.68"/>
-<wire x1="-22.86" y1="106.68" x2="-15.24" y2="106.68" width="0.1524" layer="91"/>
-</segment>
-</net>
 <net name="PA0" class="0">
 <segment>
@@
 <wire x1="142.24" y1="104.14" x2="137.16" y2="104.14" width="0.1524" layer="91"/>
 </segment>
+<segment>
+<pinref part="RPROG1" gate="G$1" pin="2"/>
+<wire x1="5.08" y1="15.24" x2="5.08" y2="12.7" width="0.1524" layer="91"/>
+</segment>
 </net>
 <net name="XBEE_RESET" class="0">
@@
 <wire x1="142.24" y1="101.6" x2="137.16" y2="101.6" width="0.1524" layer="91"/>
 </segment>
+<segment>
+<wire x1="-27.94" y1="106.68" x2="-27.94" y2="109.22" width="0.1524" layer="91"/>
+<pinref part="C1" gate="G$1" pin="1"/>
+<wire x1="-22.86" y1="106.68" x2="-27.94" y2="106.68" width="0.1524" layer="91"/>
+<wire x1="-22.86" y1="106.68" x2="-15.24" y2="106.68" width="0.1524" layer="91"/>
+<pinref part="RSENSHI" gate="G$1" pin="2"/>
+<pinref part="RSENSLO" gate="G$1" pin="1"/>
+<junction x="-27.94" y="106.68"/>
+</segment>
 </net>
 <net name="PB2" class="0">
@@
 <net name="PD5/CHGCTRL" class="0">
 <segment>
-<pinref part="PORTD" gate="G$1" pin="6"/>
-<wire x1="78.74" y1="101.6" x2="83.82" y2="101.6" width="0.1524" layer="91"/>
-</segment>
-<segment>
 <pinref part="JP2" gate="A" pin="15"/>
 <wire x1="142.24" y1="86.36" x2="137.16" y2="86.36" width="0.1524" layer="91"/>
-</segment>
-<segment>
-<pinref part="RPROG1" gate="G$1" pin="2"/>
-<wire x1="5.08" y1="15.24" x2="5.08" y2="12.7" width="0.1524" layer="91"/>
 </segment>
 </net>
@@
 </segment>
 </net>
+<net name="N$2" class="0">
+<segment>
+<pinref part="U1" gate="G$1" pin="STAT"/>
+<pinref part="LED1" gate="G$1" pin="C"/>
+</segment>
+</net>
+<net name="N$3" class="0">
+<segment>
+<pinref part="LED1" gate="G$1" pin="A"/>
+<pinref part="RSTATLED" gate="G$1" pin="1"/>
+<wire x1="-35.56" y1="15.24" x2="-35.56" y2="12.7" width="0.1524" layer="91"/>
+</segment>
+</net>
+<net name="PD5" class="0">
+<segment>
+<pinref part="PORTD" gate="G$1" pin="6"/>
+<wire x1="78.74" y1="101.6" x2="83.82" y2="101.6" width="0.1524" layer="91"/>
+</segment>
+</net>

Commit message: handle ERC
Parts:
- C2: value (none) -> 4.7uF
- C3: value (none) -> 40uF
Connections:
- removed net PD5/CHGCTRL: JP2.15
- net PD5: now also JP2.15
Changed lines of the file:
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@@
 <part name="JP3" library="pinhead" deviceset="PINHD-2X6" device="/90"/>
 <part name="GND9" library="supply1" deviceset="GND" device=""/>
-<part name="C3" library="rcl" deviceset="C-EU" device="C1210"/>
+<part name="C3" library="rcl" deviceset="C-EU" device="C1210" value="40uF"/>
 <part name="JP2" library="pinhead" deviceset="PINHD-2X8" device="/90"/>
 <part name="VREG_3.3" library="microbuilder" deviceset="LM1117" device="SOT223-WAVE"/>
@@
 <part name="+3V3" library="supply1" deviceset="+3V3" device=""/>
 <part name="+3.3V_VXMEGA" library="SparkFun-Passives" deviceset="SOLDERJUMPER" device="TRACE"/>
-<part name="C2" library="rcl" deviceset="C-EU" device="C0805K"/>
+<part name="C2" library="rcl" deviceset="C-EU" device="C0805K" value="4.7uF"/>
 <part name="U1" library="SparkFun-PowerIC" deviceset="MCP73831" device=""/>
 <part name="RPROG0" library="rcl" deviceset="R-US_" device="R0603" value="10k"/>
@@
 <wire x1="-22.86" y1="93.98" x2="-22.86" y2="99.06" width="0.1524" layer="91"/>
 <pinref part="RSENSLO" gate="G$1" pin="2"/>
+<junction x="-27.94" y="93.98"/>
 </segment>
 <segment>
@@
 <pinref part="GND9" gate="1" pin="GND"/>
 <wire x1="33.02" y1="88.9" x2="22.86" y2="88.9" width="0.1524" layer="91"/>
+<junction x="22.86" y="88.9"/>
 </segment>
 <segment>
@@
 <pinref part="VREG_3.3" gate="G$1" pin="IN"/>
 <wire x1="-5.08" y1="63.5" x2="-30.48" y2="63.5" width="0.1524" layer="91"/>
+<junction x="0" y="55.88"/>
 </segment>
 <segment>
@@
 <pinref part="RSENSLO" gate="G$1" pin="1"/>
 <junction x="-27.94" y="106.68"/>
+<junction x="-22.86" y="106.68"/>
 </segment>
 </net>
@@
 <pinref part="JP2" gate="A" pin="11"/>
 <wire x1="142.24" y1="91.44" x2="137.16" y2="91.44" width="0.1524" layer="91"/>
-</segment>
-</net>
-<net name="PD5/CHGCTRL" class="0">
-<segment>
-<pinref part="JP2" gate="A" pin="15"/>
-<wire x1="142.24" y1="86.36" x2="137.16" y2="86.36" width="0.1524" layer="91"/>
 </segment>
 </net>
@@
 <wire x1="78.74" y1="101.6" x2="83.82" y2="101.6" width="0.1524" layer="91"/>
 </segment>
+<segment>
+<pinref part="JP2" gate="A" pin="15"/>
+<wire x1="142.24" y1="86.36" x2="137.16" y2="86.36" width="0.1524" layer="91"/>
+</segment>
 </net>
 </nets>
 </sheet>
 </sheets>
+<errors>
+</errors>
 </schematic>
 </drawing>
